Commit message: Further work on moveit robai test model

File: models/robai/cyton_gamma1500.urdf (robot description, URDF)
Before this commit: robot cyton_gamma_1500, 6 links, 5 joints
Links:
- added link link7; visual box size=0.01 0.01 .5
- added link link8; visual box size=0.005 0.005 .5
Joints:
- added joint joint6: type continuous, parent link6, child link7, origin xyz=0 0 0.5 rpy=0 0 0, axis 0.0 1.0 0.0, limit lower=-0.78535 upper=0.78535 effort=1000.0 velocity=0.5
- added joint joint7: type continuous, parent link7, child link8, origin xyz=0 0 0.5 rpy=0 0 0, axis 0.0 1.0 0.0, limit lower=-0.78535 upper=0.78535 effort=1000.0 velocity=0.5
- joint joint1: limit (none) -> lower=-0.78535 upper=0.78535 effort=1000.0 velocity=0.5
- joint joint2: limit (none) -> lower=-0.78535 upper=0.78535 effort=1000.0 velocity=0.5
- joint joint3: limit (none) -> lower=-0.78535 upper=0.78535 effort=1000.0 velocity=0.5
- joint joint4: limit (none) -> lower=-0.78535 upper=0.78535 effort=1000.0 velocity=0.5
- joint joint5: limit (none) -> lower=-0.78535 upper=0.78535 effort=1000.0 velocity=0.5
