Commit message: wheelunit test xacro uses the wheelunit macro now

File: models/wheel_unit_60mm/wheel_unit_60mm.xacro (robot description, xacro)
@@ -1,232 +1,9 @@
 <robot name="wheel_unit_60mm" xmlns:xacro="http://www.ros.org/wiki/xacro">
-  <xacro:property name="wheel_base_size_x" value="0.12" />
-  <xacro:property name="wheel_base_size_y" value="0.09" />
-  <xacro:property name="wheel_base_size_z" value="0.04" />
-  <xacro:property name="wheel_base_pose_x" value="0.0" />
-  <xacro:property name="wheel_base_pose_y" value="0.0" />
-  <xacro:property name="wheel_base_pose_z" value="0.195" />
-  <xacro:property name="wheel_mount_axle_radius" value="0.0125" />
-  <xacro:property name="wheel_mount_axle_length" value="0.02" />
-  <xacro:property name="wheel_mount_axle_pose_x" value="0.04" />
-  <xacro:property name="wheel_mount_axle_pose_y" value="0.0" />
-  <xacro:property name="wheel_mount_axle_pose_z" value="0.17" />
-  <xacro:property name="wheel_horplate_size_x" value="0.14" />
-  <xacro:property name="wheel_horplate_size_y" value="0.04" />
-  <xacro:property name="wheel_horplate_size_z" value="0.005" />
-  <xacro:property name="wheel_horplate_pose_x" value="-0.05" />
-  <xacro:property name="wheel_horplate_pose_y" value="0.0" />
-  <xacro:property name="wheel_horplate_pose_z" value="-0.01" />
-  <xacro:property name="wheel_vertplate_size_x" value="0.005" />
-  <xacro:property name="wheel_vertplate_size_y" value="0.04" />
-  <xacro:property name="wheel_vertplate_size_z" value="0.12" />
-  <xacro:property name="wheel_vertplate_pose_x" value="-0.12" />
-  <xacro:property name="wheel_vertplate_pose_y" value="0.0" />
-  <xacro:property name="wheel_vertplate_pose_z" value="-0.07" />
-  <xacro:property name="wheel_axle_radius" value="0.015" />
-  <xacro:property name="wheel_axle_length" value="0.10" />
-  <xacro:property name="wheel_axle_pose_x" value="-0.07" />
-  <xacro:property name="wheel_axle_pose_y" value="0.0" />
-  <xacro:property name="wheel_axle_pose_z" value="-0.11" />
-  <xacro:property name="wheel_axle_pose_r" value="0.0" />
-  <xacro:property name="wheel_axle_pose_p" value="1.5707" />
-  <xacro:property name="wheel_axle_pose_y" value="0.0" />
-  <xacro:property name="wheel_radius" value="0.06" />
-  <xacro:property name="wheel_length" value="0.03" />
-  <xacro:property name="wheel_pose_x" value="0.02" />
-  <xacro:property name="wheel_pose_y" value="0.0" />
-  <xacro:property name="wheel_pose_z" value="0.06" />
-  <xacro:property name="wheel_pose_r" value="0.0" />
-  <xacro:property name="wheel_pose_p" value="1.5707" />
-  <xacro:property name="wheel_pose_y" value="0.0" />
-  <gazebo static="false"/>
-  <!-- wheel base -->
-  <link name='wheel_base'>
-    <collision>
-      <origin xyz="${wheel_base_pose_x} ${wheel_base_pose_y} ${wheel_base_pose_z}" rpy="0 0 0"/>
-      <geometry>
-        <box size="${wheel_base_size_x} ${wheel_base_size_x} ${wheel_base_size_x}"/>
-      </geometry>
-    </collision>
-    <inertial>
-      <origin xyz="${wheel_base_pose_x} ${wheel_base_pose_y} ${wheel_base_pose_z}" rpy="0 0 0"/>
-      <mass value="0.5"/>
-      <inertia
-        ixx="1.0" ixy="0.0" ixz="0.0"
-        iyy="1.0" iyz="0.0"
-        izz="1.0"/>
-    </inertial>
-    <visual>
-      <origin xyz="${wheel_base_pose_x} ${wheel_base_pose_y} ${wheel_base_pose_z}" rpy="0 0 0"/>
-      <geometry>
-          <box size="${wheel_base_size_x} ${wheel_base_size_y} ${wheel_base_size_z}"/>
-      </geometry>
-    </visual>
-  </link>
-  <!-- joint between wheel_base and wheel_mount_axle -->
-  <joint name="joint_base" type="fixed">
-    <parent link="wheel_base"/>
-    <child link="wheel_mount_axle"/>
-    <origin xyz="0 0 0" rpy="0 0 0"/>
-    <axis xyz="0 0 1" />
-    <dynamics damping="10.0" />
-  </joint>
-  <!-- Mount Axle -->
-  <link name="wheel_mount_axle">
-    <collision>
-      <origin xyz="${wheel_mount_axle_pose_x} ${wheel_mount_axle_pose_y} ${wheel_mount_axle_pose_z}" rpy="0 0 0"/>
-      <geometry>
-        <cylinder radius="${wheel_mount_axle_radius}" length="${wheel_mount_axle_length}"/>
-      </geometry>
-    </collision>
-    <inertial>
-      <origin xyz="${wheel_mount_axle_pose_x} ${wheel_mount_axle_pose_y} ${wheel_mount_axle_pose_z}" rpy="0 0 0"/>
-      <mass value="0.5"/>
-      <inertia
-        ixx="1.0" ixy="0.0" ixz="0.0"
-        iyy="1.0" iyz="0.0"
-        izz="1.0"/>
-    </inertial>
-    <visual>
-      <origin xyz="${wheel_mount_axle_pose_x} ${wheel_mount_axle_pose_y} ${wheel_mount_axle_pose_z}" rpy="0 0 0"/>
-      <geometry>
-        <cylinder radius="${wheel_mount_axle_radius}" length="${wheel_mount_axle_length}"/>
-      </geometry>
-    </visual>
-  </link>
-  <!-- joint between wheel_mount_axle and wheel_mount_horplate -->
-  <joint name="joint_wheel_mount_axle" type="fixed">
-    <parent link="wheel_mount_axle"/>
-    <child link="wheel_mount_horplate"/>
-    <axis xyz="0 1 0" />
-    <origin xyz="0 0 0" rpy="0 0 0"/>
-  </joint>
-  <!-- Horizontal plate -->
-  <link name="wheel_mount_horplate">
-    <collision>
-      <origin xyz="${wheel_horplate_pose_x} ${wheel_horplate_pose_y} ${wheel_horplate_pose_z}" rpy="0 0 0"/>
-      <geometry>
-        <box size="${wheel_horplate_size_x} ${wheel_horplate_size_y} ${wheel_horplate_size_z}"/>
-      </geometry>
-    </collision>
-    <inertial>
-      <origin xyz="${wheel_horplate_pose_x} ${wheel_horplate_pose_y} ${wheel_horplate_pose_z}" rpy="0 0 0"/>
-      <mass value="0.5"/>
-      <inertia
-        ixx="1.0" ixy="0.0" ixz="0.0"
-        iyy="1.0" iyz="0.0"
-        izz="1.0"/>
-    </inertial>
-    <visual>
-      <origin xyz="${wheel_horplate_pose_x} ${wheel_horplate_pose_y} ${wheel_horplate_pose_z}" rpy="0 0 0"/>
-      <geometry>
-        <box size="${wheel_horplate_size_x} ${wheel_horplate_size_y} ${wheel_horplate_size_z}"/>
-      </geometry>
-    </visual>
-  </link>
-  <!-- joint between wheel_mount_horplate and wheel_mount_vertplate -->
-  <joint name="joint_wheel_mount_vertplate" type="fixed">
-    <parent link="wheel_mount_horplate"/>
-    <child link="wheel_mount_vertplate"/>
-    <axis xyz="0 1 0" />
-    <origin xyz="0 0 0" rpy="0 0 0"/>
-  </joint>
-  <!-- Vertical plate -->
-  <link name="wheel_mount_vertplate">
-    <collision>
-      <origin xyz="${wheel_vertplate_pose_x} ${wheel_vertplate_pose_y} ${wheel_vertplate_pose_z}" rpy="0 0 0"/>
-      <geometry>
-        <box size="${wheel_vertplate_size_x} ${wheel_vertplate_size_y} ${wheel_vertplate_size_z}"/>
-      </geometry>
-    </collision>
-    <inertial>
-      <origin xyz="${wheel_vertplate_pose_x} ${wheel_vertplate_pose_y} ${wheel_vertplate_pose_z}" rpy="0 0 0"/>
-      <mass value="0.5"/>
-      <inertia
-        ixx="1.0" ixy="0.0" ixz="0.0"
-        iyy="1.0" iyz="0.0"
-        izz="1.0"/>
-    </inertial>
-    <visual>
-      <origin xyz="${wheel_vertplate_pose_x} ${wheel_vertplate_pose_y} ${wheel_vertplate_pose_z}" rpy="0 0 0"/>
-      <geometry>
-        <box size="${wheel_vertplate_size_x} ${wheel_vertplate_size_y} ${wheel_vertplate_size_z}"/>
-      </geometry>
-    </visual>
-  </link>
-  <!-- joint between wheel_mount_vertplate and wheel_axle -->
-  <joint name="joint_wheel_axle" type="fixed">
-    <parent link="wheel_mount_vertplate"/>
-    <child link="wheel_axle"/>
-    <axis xyz="0 1 0" />
-    <origin xyz="0 0 0" rpy="0 0 0"/>
-  </joint>
-  <!-- Wheel Axle -->
-  <link name="wheel_axle">
-    <collision>
-      <origin xyz="${wheel_axle_pose_x} ${wheel_axle_pose_y} ${wheel_axle_pose_z}" rpy="${wheel_axle_pose_r} ${wheel_axle_pose_p} ${wheel_axle_pose_y}"/>
-      <geometry>
-        <cylinder radius="${wheel_axle_radius}" length="${wheel_axle_length}"/>
-      </geometry>
-    </collision>
-    <inertial>
-      <origin xyz="${wheel_axle_pose_x} ${wheel_axle_pose_y} ${wheel_axle_pose_z}" rpy="${wheel_axle_pose_r} ${wheel_axle_pose_p} ${wheel_axle_pose_y}"/>
-      <mass value="0.5"/>
-      <inertia
-        ixx="1.0" ixy="0.0" ixz="0.0"
-        iyy="1.0" iyz="0.0"
-        izz="1.0"/>
-    </inertial>
-    <visual>
-      <origin xyz="${wheel_axle_pose_x} ${wheel_axle_pose_y} ${wheel_axle_pose_z}" rpy="${wheel_axle_pose_r} ${wheel_axle_pose_p} ${wheel_axle_pose_y}"/>
-      <geometry>
-        <cylinder radius="${wheel_axle_radius}" length="${wheel_axle_length}"/>
-      </geometry>
-    </visual>
-  </link>
-  <!-- joint between wheel_axle and wheel -->
-  <joint name="joint_wheel" type="continuous">
-    <parent link="wheel_axle"/>
-    <child link="wheel"/>
-    <origin xyz="0 0 0" rpy="0 0 0"/>
-    <axis xyz="1 0 0" />
-    <dynamics damping="10.0" friction="1" />
-  </joint>
-  <!-- Wheel -->
-  <link name="wheel">
-    <inertial>
-      <origin xyz="${wheel_pose_x} ${wheel_pose_y} ${wheel_pose_z}" rpy="0 0 0"/>
-      <mass value="0.5"/>
-      <inertia
-        ixx="1.0" ixy="0.0" ixz="0.0"
-        iyy="1.0" iyz="0.0"
-        izz="1.0"/>
-    </inertial>
-    <collision>
-      <origin xyz="${wheel_pose_x} ${wheel_pose_y} ${wheel_pose_z}" rpy="${wheel_pose_r} ${wheel_pose_p} ${wheel_pose_y}"/>
-      <geometry>
-        <cylinder radius="${wheel_radius}" length="${wheel_length}"/>
-      </geometry>
-     <surface>
-        <friction>
-          <ode>
-            <mu>0.85</mu>
-            <mu2>0.85</mu2>
-            <fdir1>1 1 0</fdir1>
-            <slip1>0.0</slip1>
-            <slip2>0.0</slip2>
-          </ode>
-        </friction>
-      </surface>
-    </collision>
-    <visual>
-      <origin xyz="${wheel_pose_x} ${wheel_pose_y} ${wheel_pose_z}" rpy="${wheel_pose_r} ${wheel_pose_p} ${wheel_pose_y}"/>
-      <geometry>
-        <cylinder radius="${wheel_radius}" length="${wheel_length}"/>
-      </geometry>
-    </visual>
-  </link>
-  <plugin name="wheel_unit_controller" filename="libWheelUnitController.so">
-    <caster>caster_joint</caster>
-    <wheel>wheel_joint</wheel>
-  </plugin>
+  <!-- common -->
+  <xacro:include filename="../common.xacro" />
+  <xacro:include filename="wheel_unit_60mm_macro.xacro" />
+  <xacro:wheel_unit_60mm name="test_wheel"/>
+  <gazebo>
+    <static>false</static>
+  </gazebo>
 </robot>

Commit message: Updated wheel macro

File: models/wheel_unit_60mm/wheel_unit_60mm.xacro (robot description, xacro)
@@ -3,5 +3,5 @@
   <xacro:include filename="../common.xacro" />
   <xacro:include filename="wheel_unit_60mm_macro.xacro" />
-  <xacro:wheel_unit_60mm name="test_wheel"/>
+  <xacro:wheel_unit_60mm name="test"/>
   <gazebo>
     <static>false</static>

File: models/wheel_unit_60mm/wheel_unit_60mm_macro.xacro (robot description, xacro)
@@ -42,5 +42,14 @@
   <xacro:property name="wheel_pose_p" value="0.0" />
   <xacro:property name="wheel_pose_y" value="0.0" />
-  <xacro:macro name="wheel_unit_60mm" params="name">
+  <xacro:macro name="wheel_unit_60mm" params="name parent xyz rpy">
+  	  <!-- link to parent -->
+      <joint name="${parent}_${name}_joint" type="continuous">
+	    <axis xyz="0 1 0" />
+	    <limit lower="0.0" upper="0.0" effort="7" velocity="0"/>
+	    <dynamics damping="1.0" friction="0.0" />
+	    <origin xyz="0 0 0" rpy="0 0 0" />
+	    <parent link="${parent}"/>
+	    <child link="${name}_wheel_base"/>
+	  </joint>
 	  <!-- wheel base -->
 	  <link name='${name}_wheel_base'>
