Commit message: Work on rose20.xacro model

File: models/rose20/rose20.xacro (robot description, xacro)
@@ -1,3 +1,5 @@
 <robot name="Rose20" xmlns:xacro="http://www.ros.org/wiki/xacro">
+  <xacro:include filename="../common.xacro" />
+  <xacro:include filename="../wheel_unit_60mm/wheel_unit_60mm_macro.xacro" />
   <xacro:property name="base_size_x" value="0.76" />
   <xacro:property name="base_size_y" value="0.58" />
@@ -6,5 +8,10 @@
   <xacro:property name="base_pose_y" value="0.0" />
   <xacro:property name="base_pose_z" value="0.195" />
-  <gazebo static="true"/>
+  <xacro:property name="wheel_front_x"    value="0.28" />
+  <xacro:property name="wheel_back_x"     value="-0.305" />
+  <xacro:property name="wheelbase_width"  value="0.23" />
+  <gazebo>
+    <static>false</static>
+  </gazebo>
   <!-- Used for fixing robot to Gazebo 'base_link' -->
   <link name="world"/>
@@ -35,4 +42,9 @@
     </visual>
   </link>
+  <xacro:wheel_unit_60mm name="wheel_FL"/>
+  <xacro:wheel_unit_60mm name="wheel_FR"/>
+  <xacro:wheel_unit_60mm name="wheel_BL"/>
+  <xacro:wheel_unit_60mm name="wheel_BR"/>
+<!--
   <include>
     <uri>model://wheel_unit_60mm</uri>
@@ -55,52 +67,29 @@
     <pose>-0.305 0.23 0 0 0 1.5707</pose>
   </include>
+-->
    <!-- Fix wheel units to base -->
-  <joint type="revolute" name="wheel_FL_hinge">
-    <pose>0 0 0 0 0 0</pose>
-    <child>wheel_FL::wheel_base</child>
-    <parent>base</parent>
-    <axis>
-      <xyz>0 0 0</xyz>
-      <limit>
-        <upper>0</upper>
-        <lower>0</lower>
-      </limit>
-    </axis>
-  </joint>
-  <joint type="revolute" name="wheel_FR_hinge">
-    <pose>0 0 0 0 0 0</pose>
-    <child>wheel_FR::wheel_base</child>
-    <parent>base</parent>
-    <axis>
-      <xyz>0 0 0</xyz>
-      <limit>
-        <upper>0</upper>
-        <lower>0</lower>
-      </limit>
-    </axis>
-  </joint>
-  <joint type="revolute" name="wheel_BL_hinge">
-    <pose>0 0 0 0 0 0</pose>
-    <child>wheel_BL::wheel_base</child>
-    <parent>base</parent>
-    <axis>
-      <xyz>0 0 0</xyz>
-      <limit>
-        <upper>0</upper>
-        <lower>0</lower>
-      </limit>
-    </axis>
-  </joint>
-  <joint type="revolute" name="wheel_BR_hinge">
-    <pose>0 0 0 0 0 0</pose>
-    <child>wheel_BR::wheel_base</child>
-    <parent>base</parent>
-    <axis>
-      <xyz>0 0 0</xyz>
-      <limit>
-        <upper>0</upper>
-        <lower>0</lower>
-      </limit>
-    </axis>
+  <joint name="joint_wheel_axle" type="fixed">
+    <parent link="base"/>
+    <child link="wheel_FL_wheel_base"/>
+    <axis xyz="0 1 0" />
+    <origin xyz="${wheel_front_x} ${-wheelbase_width} 0" rpy="0 0 -${pi/2}"/>
+  </joint>
+  <joint name="joint_wheel_axle" type="fixed">
+    <parent link="base"/>
+    <child link="wheel_FR_wheel_base"/>
+    <axis xyz="0 1 0" />
+    <origin xyz="${wheel_front_x} ${wheelbase_width} 0" rpy="0 0 ${pi/2}"/>
+  </joint>
+  <joint name="joint_wheel_axle" type="fixed">
+    <parent link="base"/>
+    <child link="wheel_BL_wheel_base"/>
+    <axis xyz="0 1 0" />
+    <origin xyz="${wheel_back_x} ${-wheelbase_width} 0" rpy="0 0 -${pi/2}"/>
+  </joint>
+  <joint name="joint_wheel_axle" type="fixed">
+    <parent link="base"/>
+    <child link="wheel_BR_wheel_base"/>
+    <axis xyz="0 1 0" />
+    <origin xyz="${wheel_back_x} ${wheelbase_width} 0" rpy="0 0 ${pi/2}"/>
   </joint>
   <!-- Lift mid-->
@@ -528,5 +517,4 @@
   </joint>
   <plugin name="NeckController" filename="libNeckController.so"/>
-  </plugin>
   <!-- END kinect -->
   <!-- START Hokuyo -->

Commit message: Rose sim base plus wheels working

File: models/rose20/rose20.xacro (robot description, xacro)
@@ -7,5 +7,5 @@
   <xacro:property name="base_pose_x" value="0.0" />
   <xacro:property name="base_pose_y" value="0.0" />
-  <xacro:property name="base_pose_z" value="0.195" />
+  <xacro:property name="base_pose_z" value="0.2" />
   <xacro:property name="wheel_front_x"    value="0.28" />
   <xacro:property name="wheel_back_x"     value="-0.305" />
@@ -14,524 +14,13 @@
     <static>false</static>
   </gazebo>
-  <!-- Used for fixing robot to Gazebo 'base_link' -->
-  <link name="world"/>
-  <joint name="fixed" type="fixed">
-    <parent link="world"/>
-    <child link="base"/>
-  </joint>
   <link name='base'>
-    <collision name='base_collision'>
-      <origin xyz="${base_pose_x} ${base_pose_y} ${base_pose_z}" rpy="0 0 0"/>
-      <geometry>
-          <box size="${base_size_x} ${base_size_x} ${base_size_x}"/>
-      </geometry>
-    </collision>
-    <inertial>
-      <origin xyz="${base_pose_x} ${base_pose_y} ${base_pose_z}" rpy="0 0 0"/>
-      <mass>30.0</mass>
-      <inertia
-        ixx="1.0" ixy="0.0" ixz="0.0"
-        iyy="1.0" iyz="0.0"
-        izz="1.0"/>
-    </inertial>
-    <visual name='base_visual'>
-      <origin xyz="${base_pose_x} ${base_pose_y} ${base_pose_z}" rpy="0 0 0"/>
-      <geometry>
-         <box size="${base_size_x} ${base_size_x} ${base_size_x}"/>
-      </geometry>
-    </visual>
+    <xacro:default_box  xyz=  "${base_pose_x} ${base_pose_y} ${base_pose_z}"
+                        rpy=  "0 0 0"
+                        size= "${base_size_x} ${base_size_y} ${base_size_z}"/>
+    <xacro:default_inertial mass="30.0"/>
   </link>
-  <xacro:wheel_unit_60mm name="wheel_FL"/>
-  <xacro:wheel_unit_60mm name="wheel_FR"/>
-  <xacro:wheel_unit_60mm name="wheel_BL"/>
-  <xacro:wheel_unit_60mm name="wheel_BR"/>
-<!--
-  <include>
-    <uri>model://wheel_unit_60mm</uri>
-    <name>wheel_FL</name>
-    <pose>0.28 -0.23 0 0 0 -1.5707</pose>
-  </include>
-  <include>
-    <uri>model://wheel_unit_60mm</uri>
-    <name>wheel_FR</name>
-    <pose>0.28 0.23 0 0 0 1.5707</pose>
-  </include>
-  <include>
-    <uri>model://wheel_unit_60mm</uri>
-    <name>wheel_BL</name>
-    <pose>-0.305 -0.23 0 0 0 -1.5707</pose>
-  </include>
-  <include>
-    <uri>model://wheel_unit_60mm</uri>
-    <name>wheel_BR</name>
-    <pose>-0.305 0.23 0 0 0 1.5707</pose>
-  </include>
--->
-   <!-- Fix wheel units to base -->
-  <joint name="joint_wheel_axle" type="fixed">
-    <parent link="base"/>
-    <child link="wheel_FL_wheel_base"/>
-    <axis xyz="0 1 0" />
-    <origin xyz="${wheel_front_x} ${-wheelbase_width} 0" rpy="0 0 -${pi/2}"/>
-  </joint>
-  <joint name="joint_wheel_axle" type="fixed">
-    <parent link="base"/>
-    <child link="wheel_FR_wheel_base"/>
-    <axis xyz="0 1 0" />
-    <origin xyz="${wheel_front_x} ${wheelbase_width} 0" rpy="0 0 ${pi/2}"/>
-  </joint>
-  <joint name="joint_wheel_axle" type="fixed">
-    <parent link="base"/>
-    <child link="wheel_BL_wheel_base"/>
-    <axis xyz="0 1 0" />
-    <origin xyz="${wheel_back_x} ${-wheelbase_width} 0" rpy="0 0 -${pi/2}"/>
-  </joint>
-  <joint name="joint_wheel_axle" type="fixed">
-    <parent link="base"/>
-    <child link="wheel_BR_wheel_base"/>
-    <axis xyz="0 1 0" />
-    <origin xyz="${wheel_back_x} ${wheelbase_width} 0" rpy="0 0 ${pi/2}"/>
-  </joint>
-  <!-- Lift mid-->
-  <link name='lift_mid'>
-    <pose> 0.20 0 0.361 0 0.785 0</pose>
-    <inertial>
-      <pose> 0 0 0 0 0 0</pose>
-      <mass>0.5</mass>
-    </inertial>
-    <collision name='lift_mid_collision'>
-      <geometry>
-        <box>
-          <size>0.41 0.115 0.05</size>
-        </box>
-      </geometry>
-    </collision>
-    <visual name='lift_mid_visual'>
-      <geometry>
-        <box>
-          <size>0.41 0.115 0.05</size>
-        </box>
-      </geometry>
-    </visual>
- </link>
- <!-- lift left -->
-  <link name='lift_left'>
-    <pose> 0.06 0.24 0.361 0 0.785 0</pose>
-    <inertial>
-      <pose> 0 0 0 0 0 0</pose>
-      <mass>0.5</mass>
-    </inertial>
-    <collision name='lift_left_collision'>
-      <geometry>
-        <box>
-          <size>0.41 0.09 0.05</size>
-        </box>
-      </geometry>
-    </collision>
-    <visual name='lift_left_visual'>
-      <geometry>
-        <box>
-          <size>0.41 0.09 0.05</size>
-        </box>
-      </geometry>10.000
-    </visual>
-  </link>
- <!-- lift right -->
- <link name='lift_right'>
-    <pose> 0.06 -0.24 0.361 0 0.785 0</pose>
-    <inertial>
-      <pose> 0 0 0 0 0 0</pose>
-      <mass>0.5</mass>
-    </inertial>
-    <collision name='lift_right_collision'>
-      <geometry>
-        <box>
-          <size>0.41 0.09 0.05</size>
-        </box>
-      </geometry>
-    </collision>
-    <visual name='lift_right_visual'>
-      <geometry>
-        <box>
-          <size>0.41 0.09 0.05</size>
-        </box>
-      </geometry>
-    </visual>
-  </link>
-  <!-- lift top -->
- <link name='lift_top'>
-    <pose> -0.06 0 0.55 0 0 0</pose>
-    <inertial>
-      <pose> 0 0 0 0 0 0</pose>
-      <mass>30.0</mass>
-    </inertial>
-    <collision name='lift_top_bar_collision'>
-      <geometry>
-        <box>
-          <size>0.06 0.56 0.06</size>
-        </box>
-      </geometry>
-    </collision>
-    <visual name='lift_top_bar_visual'>
-      <geometry>
-        <box>
-          <size>0.06 0.56 0.06</size>
-        </box>
-      </geometry>
-    </visual>
-    <collision name='lift_top_collision'>
-      <pose> 0 0 0.285 0 0 0</pose>
-      <geometry>
-        <box>
-          <size>0.29 0.24 0.57</size>
-        </box>
-      </geometry>
-    </collision>
-    <visual name='lift_top_visual'>
-      <pose> 0 0 0.285 0 0 0</pose>
-      <geometry>
-        <box>
-          <size>0.29 0.24 0.57</size>
-        </box>
-      </geometry>
-    </visual>
-  </link>
-  <!-- Lift joints -->
-  <joint type="revolute" name="lift_mid_bottom_hinge">
-    <pose>0.19 0.0 0 0 0 0</pose>
-    <child>lift_mid</child>
-    <parent>base</parent>
-    <axis>
-      <xyz>0 1 0</xyz>
-      <limit>
-        <upper>0.785</upper>
-        <lower>-0.785</lower>
-      </limit>
-      <dynamics>
-        <damping>1</damping>
-        <friction>1</friction>
-      </dynamics>
-    </axis>
-  </joint>
-  <joint type="revolute" name="lift_mid_top_hinge">
-    <pose>-0.19 0.0 0 0 0 0</pose>
-    <child>lift_mid</child>
-    <parent>lift_top</parent>
-    <axis>
-      <xyz>0 1 0</xyz>
-      <limit>
-        <upper>0.785</upper>
-        <lower>-0.785</lower>
-      </limit>
-      <dynamics>
-        <damping>1</damping>
-        <friction>1</friction>
-      </dynamics>
-    </axis>
-  </joint>
-  <joint type="revolute" name="lift_left_bottom_hinge">
-    <pose>0.19 0 0 0 0 0</pose>
-    <child>lift_left</child>
-    <parent>base</parent>
-    <axis>
-      <xyz>0 1 0</xyz>
-      <limit>
-        <upper>0.785</upper>
-        <lower>-0.785</lower>
-      </limit>
-      <dynamics>
-        <damping>1</damping>
-        <friction>1</friction>
-      </dynamics>
-    </axis>
-  </joint>
-  <joint type="revolute" name="lift_left_top_hinge">
-    <pose>-0.19 0 0 0 0 0</pose>
-    <child>lift_left</child>
-    <parent>lift_top</parent>
-    <axis>
-      <xyz>0 1 0</xyz>
-      <limit>
-        <upper>0.785</upper>
-        <lower>-0.785</lower>
-      </limit>
-      <dynamics>
-        <damping>1</damping>
-        <friction>1</friction>
-      </dynamics>
-    </axis>
-  </joint>
-  <joint type="revolute" name="lift_right_bottom_hinge">
-    <pose>0.19 0 0 0 0 0</pose>
-    <child>lift_right</child>
-    <parent>base</parent>
-    <axis>
-      <xyz>0 1 0</xyz>
-      <limit>
-        <upper>0.785</upper>
-        <lower>-0.785</lower>
-      </limit>
-      <dynamics>
-        <damping>1</damping>
-        <friction>1</friction>
-      </dynamics>
-    </axis>
-  </joint>
-  <joint type="revolute" name="lift_right_top_hinge">
-    <pose>-0.19 0 0 0 0 0</pose>
-    <child>lift_right</child>
-    <parent>lift_top</parent>
-    <axis>
-      <xyz>0 1 0</xyz>
-      <limit>
-        <upper>0.785</upper>
-        <lower>-0.785</lower>
-      </limit>
-      <dynamics>
-        <damping>1</damping>
-        <friction>1</friction>
-      </dynamics>
-    </axis>
-  </joint>
-  <!-- START base -> lift mechanism -->
-  <link name='base_lift_axle'>
-    <pose> -0.14 0 0.155 0 1.5707 1.5707</pose>
-    <collision name='base_lift_axle_collision'>
-      <geometry>
-        <cylinder>
-          <radius>.02</radius>
-          <length>.19</length>
-        </cylinder>
-      </geometry>
-    </collision>
-    <visual name='base_lift_axle_visual'>
-      <geometry>
-        <cylinder>
-          <radius>.02</radius>
-          <length>.19</length>
-        </cylinder>
-      </geometry>
-    </visual>
-  </link>
-  <link name='lift_lift_axle'>
-    <pose> 0.30 0 0.155 0 1.5707 1.5707</pose>
-    <collision name='lift_lift_axle_collision'>
-      <geometry>
-        <cylinder>
-          <radius>.02</radius>
-          <length>.19</length>
-        </cylinder>
-      </geometry>
-    </collision>
-    <visual name='lift_lift_axle_visual'>
-      <geometry>
-        <cylinder>
-          <radius>.02</radius>
-          <length>.19</length>
-        </cylinder>
-      </geometry>
-    </visual>
-  </link>
-  <joint type="revolute" name="base_lift_axle_hinge">
-    <pose>0 0 0 0 0 0</pose>
-    <child>base_lift_axle</child>
-    <parent>base</parent>
-    <axis>
-      <xyz>0 1 0</xyz>
-    </axis>
-  </joint>
-  <joint type="revolute" name="lift_lift_axle_hinge">
-    <pose>0 0 0 0 0 0</pose>
-    <child>lift_lift_axle</child>
-    <parent>lift_mid</parent>
-    <axis>
-      <xyz>0 1 0</xyz>
-    </axis>
-  </joint>
-  <joint type="prismatic" name="base_lift_prismatic">
-    <pose>0 0 0 0 0 0</pose>
-    <child>lift_lift_axle</child>
-    <parent>base_lift_axle</parent>
-    <axis>
-      <xyz>1 0 0</xyz>
-      <!--<limit>
-        <upper>0.02</upper>
-        <lower>-0.02</lower>
-      </limit> -->
-      <dynamics>
-        <damping>100000</damping>
-        <friction>1000000</friction>
-      </dynamics>
-    </axis>
-  </joint>
-  <plugin name="LiftController" filename="libLiftController.so"/>
-  <!-- END base -> lift mechanism -->
-  <!-- START neck -->
-  <link name='neck_pan'>
-    <pose> 0 0 1.59 0 0.0 0</pose>
-    <inertial>
-      <pose> 0 0 0 0 0 0</pose>
-      <mass>0.25</mass>
-    </inertial>
-    <collision name='neck_pan_collision'>
-      <pose>0 0 0 0 0 0</pose>
-      <geometry>
-        <box>
-          <size>0.05 0.03 0.04</size>
-        </box>
-      </geometry>
-    </collision>
-    <visual name='neck_pan_visual'>
-      <pose>0 0 0 0 0 0</pose>
-      <geometry>
-        <box>
-          <size>0.05 0.03 0.04</size>
-        </box>
-      </geometry>
-    </visual>
-  </link>
-  <link name='neck_tilt'>
-    <pose> 0 0 1.6375 0 0.0 0</pose>
-    <inertial>
-      <pose> 0 0 0 0 0 0</pose>
-      <mass>0.25</mass>
-    </inertial>
-    <collision name='neck_tilt_collision'>
-      <pose>0 0 0 0 0 0</pose>
-      <geometry>
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
File: models/wheel_unit_60mm/wheel_unit_60mm_macro.xacro (robot description, xacro)
@@ -43,14 +43,11 @@
   <xacro:property name="wheel_pose_y" value="0.0" />
   <xacro:macro name="wheel_unit_60mm" params="name parent xyz rpy">
-  	  <!-- link to parent -->
-      <joint name="${parent}_${name}_joint" type="continuous">
-	    <axis xyz="0 1 0" />
-	    <limit lower="0.0" upper="0.0" effort="7" velocity="0"/>
-	    <dynamics damping="1.0" friction="0.0" />
-	    <origin xyz="0 0 0" rpy="0 0 0" />
+  	  <!-- link to parent
+      <joint name="${parent}_${name}_joint" type="fixed">
+	    <axis xyz="0 1 0"/>
+	    <origin xyz="${xyz}" rpy="${rpy}" />
 	    <parent link="${parent}"/>
 	    <child link="${name}_wheel_base"/>
 	  </joint>
-	  <!-- wheel base -->
 	  <link name='${name}_wheel_base'>
 	    <xacro:default_box  xyz=  "0 0 ${wheel_mount_axle_length/2 + wheel_base_size_z/2}"
@@ -58,12 +55,12 @@
 	                        size= "${wheel_base_size_x} ${wheel_base_size_y} ${wheel_base_size_z}"/>
 	    <xacro:default_inertial mass="0.5"/>
-	  </link>
-	  <!-- joint between wheel_base and wheel_mount_axle -->
-	  <joint name="${name}_joint_base" type="revolute">
-	    <parent link="${name}_wheel_base"/>
+	  </link>-->
+	  <!-- joint between parent and wheel_mount_axle -->
+	  <joint name="${name}_joint_caster" type="revolute">
+	    <parent link="${parent}"/>
 	    <child link="${name}_wheel_mount_axle"/>
-	    <origin xyz="${wheel_base_size_x/2 - wheel_mount_axle_radius - 0.01} 0 0" rpy="0 0 0"/>
+	    <origin xyz="${xyz}" rpy="${rpy}"/>
 	    <axis xyz="0 0 1" />
-	    <dynamics damping="10.0" friction="1.0"/>
+	    <dynamics damping="1.0" friction="0.0"/>
 	    <limit effort="10.0" lower="${-wheel_base_angle}" upper="${wheel_base_angle}" velocity="0.5"/>
 	  </joint>
@@ -135,15 +132,4 @@
 	        <cylinder radius="${wheel_radius}" length="${wheel_length}"/>
 	      </geometry>
-	      <surface>
-	        <friction>
-	          <ode>
-	            <mu>0.85</mu>
-	            <mu2>0.85</mu2>
-	            <fdir1>1 1 0</fdir1>
-	            <slip1>0.0</slip1>
-	            <slip2>0.0</slip2>
-	          </ode>
-	        </friction>
-	      </surface>
 	    </collision>
 	    <visual>
@@ -154,7 +140,12 @@
 	    </visual>
 	  </link>
+	  <gazebo reference="${name}_wheel">
+	    <mu1>0.850000</mu1>
+        <mu2>0.850000</mu2>
+        <fdir1>1.000000 1.000000 0.000000</fdir1>
+	  </gazebo>
 	  <gazebo >
 	    <plugin name="${name}_wheel_unit_controller" filename="libWheelUnitController.so">
-	      <caster>${name}_joint_base</caster>
+	      <caster>${name}_joint_caster</caster>
 	      <wheel>${name}_joint_wheel</wheel>
 	    </plugin>
