Commit message: Work on models and controllers

File: models/rose20/rose20.xacro (robot description, xacro)
@@ -11,4 +11,29 @@
   <xacro:property name="wheel_back_x"     value="-0.305" />
   <xacro:property name="wheelbase_width"  value="0.23" />
+  <xacro:property name="liftmid_size_x" value="0.41" />
+  <xacro:property name="liftmid_size_y" value="0.115" />
+  <xacro:property name="liftmid_size_z" value="0.05" />
+  <xacro:property name="liftmid_pose_x" value="-0.205" />
+  <xacro:property name="liftmid_pose_y" value="0.0" />
+  <xacro:property name="liftmid_pose_z" value="0.0" />
+  <xacro:property name="liftsides_size_x" value="0.41" />
+  <xacro:property name="liftsides_size_y" value="0.09" />
+  <xacro:property name="liftsides_size_z" value="0.05" />
+  <xacro:property name="liftsides_pose_x" value="-0.345" />
+  <xacro:property name="liftsides_pose_y" value="0.24" />
+  <xacro:property name="liftsides_pose_z" value="0.0"/>
+  <xacro:property name="lifttopbar_size_x" value="0.06" />
+  <xacro:property name="lifttopbar_size_y" value="0.56" />
+  <xacro:property name="lifttopbar_size_z" value="0.06" />
+  <xacro:property name="lifttopbar_pose_x" value="-0.06" />
+  <xacro:property name="lifttopbar_pose_y" value="0.0" />
+  <xacro:property name="lifttopbar_pose_z" value="0.55"/>
+  <xacro:property name="lifttopbox_size_x" value="0.29" />
+  <xacro:property name="lifttopbox_size_y" value="0.24" />
+  <xacro:property name="lifttopbox_size_z" value="0.57" />
+  <xacro:property name="lifttopbox_pose_x" value="0.0" />
+  <xacro:property name="lifttopbox_pose_y" value="0.0" />
+  <xacro:property name="lifttopbox_pose_z" value="0.285"/>
+  <xacro:property name="lift_rpy" value="0 0 0"/>
   <gazebo>
     <static>false</static>
@@ -20,7 +45,110 @@
     <xacro:default_inertial mass="30.0"/>
   </link>
+  <!-- Wheel units -->
   <xacro:wheel_unit_60mm name="wheel_FL" parent="base" xyz="${wheel_front_x} ${-wheelbase_width} ${base_pose_z - base_size_z/2}" rpy="0 0 ${-pi/2}"/>
   <xacro:wheel_unit_60mm name="wheel_FR" parent="base" xyz="${wheel_front_x} ${wheelbase_width}  ${base_pose_z - base_size_z/2}" rpy="0 0 ${pi/2}"/>
   <xacro:wheel_unit_60mm name="wheel_BL" parent="base" xyz="${wheel_back_x}  ${-wheelbase_width} ${base_pose_z - base_size_z/2}" rpy="0 0 ${-pi/2}"/>
   <xacro:wheel_unit_60mm name="wheel_BR" parent="base" xyz="${wheel_back_x}  ${wheelbase_width}  ${base_pose_z - base_size_z/2}" rpy="0 0 ${pi/2}"/>
+  <!-- joint between base and lift_mid -->
+  <joint name="lift_mid_bottom_joint" type="revolute">
+    <parent link="base"/>
+    <child link="lift_mid"/>
+    <axis xyz="0 1 0" />
+    <origin xyz="${base_size_x/2 - 0.055} 0 ${base_pose_z}" rpy="0 0 0"/>
+    <dynamics damping="1.0" friction="1.0"/>
+    <limit effort="10.0" lower="0.0" upper="${pi/2}" velocity="1.0"/>
+  </joint>
+  <!-- Lift mid-->
+  <link name='lift_mid'>
+    <xacro:default_box  xyz=  "${liftmid_pose_x} ${liftmid_pose_y} ${liftmid_pose_z}"
+                        rpy=  "${lift_rpy}"
+                        size= "${liftmid_size_x} ${liftmid_size_y} ${liftmid_size_z}"/>
+    <xacro:default_inertial mass="0.5"/>
+  </link>
+  <!-- joint between base and lift_left -->
+  <!-- URDF DOES NOT SUPPORT JOINT LOOPS SO ONLY USE ONE BAR OF THE LIFFT FOR NOW
+  <joint name="lift_left_bottom_joint" type="revolute">
+    <parent link="base"/>
+    <child link="lift_left"/>
+    <axis xyz="0 1 0" />
+    <origin xyz="${base_size_x/2 - 0.055 - 0.14} ${liftsides_pose_y} ${base_pose_z}" rpy="0 0 0"/>
+    <dynamics damping="1.0" friction="1.0"/>
+    <limit effort="10.0" lower="0.0" upper="${pi/2}" velocity="1.0"/>
+  </joint>
+  -->
+  <!-- lift left -->
+  <!-- URDF DOES NOT SUPPORT JOINT LOOPS SO ONLY USE ONE BAR OF THE LIFFT FOR NOW
+  <link name='lift_left'>
+    <xacro:default_box  xyz=  "${-liftsides_size_x/2} 0 0"
+                        rpy=  "0 0 0"
+                        size= "${liftsides_size_x} ${liftsides_size_y} ${liftsides_size_z}"/>
+    <xacro:default_inertial mass="0.5"/>
+  </link>
+  -->
+  <!-- joint between base and lift_right -->
+  <!-- URDF DOES NOT SUPPORT JOINT LOOPS SO ONLY USE ONE BAR OF THE LIFFT FOR NOW
+  <joint name="lift_right_bottom_joint" type="revolute">
+    <parent link="base"/>
+    <child link="lift_right"/>
+    <axis xyz="0 1 0" />
+    <origin xyz="${base_size_x/2 - 0.055 - 0.14} ${-liftsides_pose_y} ${base_pose_z}" rpy="0 0 0"/>
+    <dynamics damping="1.0" friction="1.0"/>
+    <limit effort="10.0" lower="0.0" upper="${pi/2}" velocity="1.0"/>
+  </joint>
+  -->
+  <!-- lift right -->
+  <!-- URDF DOES NOT SUPPORT JOINT LOOPS SO ONLY USE ONE BAR OF THE LIFFT FOR NOW
+  <link name='lift_right'>
+      <xacro:default_box xyz=  "${-liftsides_size_x/2} 0 0"
+                          rpy=  "0 0 0"
+                          size= "${liftsides_size_x} ${liftsides_size_y} ${liftsides_size_z}"/>
+     <xacro:default_inertial mass="0.5"/>
+  </link>
+  -->
+  <!-- macro for joining the lift bars to the top of rose -->
+  <xacro:macro name="lift_bar_joint" params="parent">
+    <joint name="${parent}_box_joint" type="continuous">
+      <parent link="${parent}"/>
+      <child link="lift_top_box"/>
+      <axis xyz="0 1 0" />
+      <origin xyz="${-liftsides_size_x} 0 0" rpy="0 0 0"/>
+      <dynamics damping="1.0" friction="1.0"/>
+      <limit effort="10.0" lower="0" upper="0" velocity="1.0"/>
+    </joint>
+  </xacro:macro>
+  <!-- lift top box -->
+  <link name='lift_top_box'>
+    <xacro:default_box  xyz=  "-0.10 0 ${lifttopbox_size_z/2}"
+                        rpy=  "0 0 0"
+                        size= "${lifttopbox_size_x} ${lifttopbox_size_y} ${lifttopbox_size_z}"/>
+    <xacro:default_inertial mass="0.1"/>
+  </link>
+  <!-- joint between lift_mid and lift_top_box-->
+  <xacro:lift_bar_joint parent="lift_mid"/>
+  <!-- URDF DOES NOT SUPPORT JOINT LOOPS SO ONLY USE ONE BAR OF THE LIFFT FOR NOW
+  <xacro:lift_bar_joint parent="lift_left"/>
+  <xacro:lift_bar_joint parent="lift_right"/>
+  -->
+  <!-- joint between lift_top_box and lift_top_bar -->
+  <joint name="lift_mid_top_joint" type="revolute">
+    <parent link="lift_top_box"/>
+    <child link="lift_top_bar"/>
+    <axis xyz="0 1 0" />
+    <origin xyz="-0.14 0 0" rpy="0 0 0"/>
+    <dynamics damping="0.0" friction="0.0"/>
+    <limit effort="0.0" lower="${-pi/2}" upper="0.0" velocity="0.0"/>
+  </joint>
+  <!-- lift top bar -->
+  <link name='lift_top_bar'>
+    <xacro:default_box  xyz=  "0 0 0"
+                        rpy=  "0 0 0"
+                        size= "${lifttopbar_size_x} ${lifttopbar_size_y} ${lifttopbar_size_z}"/>
+    <xacro:default_inertial mass="1.0"/>
+  </link>
+  <gazebo>
+    <plugin name="LiftController" filename="libLiftController.so">
+      <bottom_lift_joint>lift_mid_bottom_joint</bottom_lift_joint>
+      <top_lift_joint>lift_mid_box_joint</top_lift_joint>
+    </plugin>
+  </gazebo>
 </robot>
