Commit message: Wheelunit naming

File: src/rose20_description/rose20/rose20.xacro (robot description, xacro)
@@ -70,8 +70,8 @@
   </link>
   <!-- Wheel units -->
-  <xacro:wheel_unit_60mm name="wheel_FL" parent="base" xyz="${wheel_front_x} ${-wheelbase_width} ${base_pose_z - base_size_z/2}" rpy="0 0 ${-pi/2}"/>
-  <xacro:wheel_unit_60mm name="wheel_FR" parent="base" xyz="${wheel_front_x} ${wheelbase_width}  ${base_pose_z - base_size_z/2}" rpy="0 0 ${pi/2}"/>
-  <xacro:wheel_unit_60mm name="wheel_BL" parent="base" xyz="${wheel_back_x}  ${-wheelbase_width} ${base_pose_z - base_size_z/2}" rpy="0 0 ${-pi/2}"/>
-  <xacro:wheel_unit_60mm name="wheel_BR" parent="base" xyz="${wheel_back_x}  ${wheelbase_width}  ${base_pose_z - base_size_z/2}" rpy="0 0 ${pi/2}"/>
+  <xacro:wheel_unit_60mm name="FL" parent="base" xyz="${wheel_front_x} ${-wheelbase_width} ${base_pose_z - base_size_z/2}" rpy="0 0 ${-pi/2}"/>
+  <xacro:wheel_unit_60mm name="FR" parent="base" xyz="${wheel_front_x} ${wheelbase_width}  ${base_pose_z - base_size_z/2}" rpy="0 0 ${pi/2}"/>
+  <xacro:wheel_unit_60mm name="BL" parent="base" xyz="${wheel_back_x}  ${-wheelbase_width} ${base_pose_z - base_size_z/2}" rpy="0 0 ${-pi/2}"/>
+  <xacro:wheel_unit_60mm name="BR" parent="base" xyz="${wheel_back_x}  ${wheelbase_width}  ${base_pose_z - base_size_z/2}" rpy="0 0 ${pi/2}"/>
   <!-- joint between base and lift_mid -->
   <joint name="lift_mid_bottom_joint" type="revolute">

File: src/rose20_description/wheel_unit_60mm/wheel_unit_60mm_macro.xacro (robot description, xacro)
@@ -57,5 +57,5 @@
 	  </link>-->
 	  <!-- joint between parent and wheel_mount_axle -->
-	  <joint name="${name}_joint_caster" type="revolute">
+	  <joint name="${name}_caster" type="revolute">
 	    <parent link="${parent}"/>
 	    <child link="${name}_wheel_mount_axle"/>
@@ -117,5 +117,5 @@
 	  </link>
 	  <!-- joint between wheel_axle and wheel -->
-	  <joint name="${name}_joint_wheel" type="continuous">
+	  <joint name="${name}_wheel" type="continuous">
 	    <parent link="${name}_wheel_axle"/>
 	    <child link="${name}_wheel"/>
@@ -147,6 +147,6 @@
 	  <gazebo >
 	    <plugin name="${name}_wheel_unit_controller" filename="libWheelUnitController.so">
-	      <caster>${name}_joint_caster</caster>
-	      <wheel>${name}_joint_wheel</wheel>
+	      <caster>${name}_caster</caster>
+	      <wheel>${name}_wheel</wheel>
 	    </plugin>
 	  </gazebo>
