Commit message: Robai arm model angles fix

File: src/rose20_description/cyton_gamma_1500/new/urdf/arm/arm.urdf.xacro (robot description, xacro)
@@ -67,5 +67,5 @@
                   <limit lower="0" upper="0" effort="0" velocity="0"/>
                   <limit lower="-${M_PI/2}" upper="${M_PI/2}" effort="1000" velocity="1000"/>
-                  <origin xyz="0 ${j1_radius + (j2_h /2)} 0" rpy="-${M_PI/2} 0 0"/>
+                  <origin xyz="0 ${j1_radius + (j2_h /2)} 0" rpy="-${M_PI/2} -${M_PI} 0"/>
                   <origin xyz="0 0 ${(j2_h/2) + j2_radius}" rpy="0 ${M_PI/2} 0"/>
   </xacro:joint_arm>
@@ -81,5 +81,5 @@
                   <limit lower="-${M_PI/2}" upper="${M_PI/2}" effort="1000" velocity="1000"/>
                   <origin xyz="-${j2_radius + (j3_h /2)} 0 0" rpy="0 -${M_PI/2} 0"/>
-                  <origin xyz="0 0 ${(j3_h/2) + j3_radius}" rpy="${M_PI/2} 0 0"/>
+                  <origin xyz="0 0 ${(j3_h/2) + j3_radius}" rpy="${M_PI/2} 0 ${M_PI}"/>
   </xacro:joint_arm>
   <xacro:joint_arm
@@ -93,5 +93,5 @@
                   <limit lower="0" upper="0" effort="0" velocity="0"/>
                   <limit lower="-${M_PI/2}" upper="${M_PI/2}" effort="1000" velocity="1000"/>
-                  <origin xyz="0 ${j3_radius + (j4_h /2)} 0" rpy="-${M_PI/2} 0 0"/>
+                  <origin xyz="0 ${j3_radius + (j4_h /2)} 0" rpy="-${M_PI/2} -${M_PI} 0"/>
                   <origin xyz="0 0 ${(j4_h/2) + j4_radius}" rpy="0 ${M_PI/2} 0"/>
   </xacro:joint_arm>
@@ -107,5 +107,5 @@
                   <limit lower="-${M_PI/2}" upper="${M_PI/2}" effort="1000" velocity="1000"/>
                   <origin xyz="-${j4_radius + (j5_h /2)} 0 0" rpy="0 -${M_PI/2} 0"/>
-                  <origin xyz="0 0 ${(j5_h/2) + j5_radius}" rpy="${M_PI/2} 0 0"/>
+                  <origin xyz="0 0 ${(j5_h/2) + j5_radius}" rpy="${M_PI/2} 0 ${M_PI}"/>
   </xacro:joint_arm>
  </xacro:macro>

File: src/rose20_description/cyton_gamma_1500/new/urdf/gripper/gripper.urdf.xacro (robot description, xacro)
@@ -29,5 +29,5 @@
                   parent=     "arm_link_cyl_5"
                   type =      "revolute">
-                  <origin xyz="0 ${j5_radius + (gr1_1 /2)} 0" rpy="-${M_PI/2} 0 0"/>
+                  <origin xyz="0 ${j5_radius + (gr1_1 /2)} 0" rpy="-${M_PI/2} ${M_PI/2} 0"/>
  		  <limit lower="-${M_PI}" upper="${M_PI}" effort="1000" velocity="1000"/>
                   <box size ="${gr1_1} ${gr1_1} ${gr1_1}" />

Commit message: Stuff
Former-commit-id: 599b82b0c8838fbcbb757abcf4d1568afcaf5d9d

File: src/rose20_description/cyton_gamma_1500/new/urdf/arm/arm.urdf.xacro (robot description, xacro)
@@ -2,5 +2,5 @@
 <robot xmlns:xacro="http://ros.org/wiki/xacro">
  <xacro:include filename="$(find rose20_description)/cyton_gamma_1500/new/urdf/properties/properties.urdf.xacro" />
- <xacro:macro name="joint_arm" params="suffix radius length parent type_box type_cyl *size *limit_box *limit_cyl *origin_box *origin_cyl">
+ <xacro:macro name="joint_arm" params="suffix radius length parent type_box type_cyl *size *limit_box *limit_cyl *origin_box *origin_cyl *axis_box *axis_cyl">
   <!--Part 1: box -->
   <joint name="arm_joint_box_${suffix}" type="${type_box}" >
@@ -8,5 +8,5 @@
     <child link="arm_link_box_${suffix}" />
      <insert_block name="limit_box"/>
-    <axis xyz="0 0 1"/>
+     <insert_block name="axis_box"/>
      <insert_block name="origin_box"/>
   </joint>
@@ -26,6 +26,6 @@
     <parent link="arm_link_box_${suffix}" />
     <child link="arm_link_cyl_${suffix}" />
-     <insert_block name="limit_cyl"/>
-    <axis xyz="0 0 1"/>
+    <insert_block name="limit_cyl"/>
+    <insert_block name="axis_cyl"/>
     <insert_block name="origin_cyl"/>
   </joint>
@@ -53,7 +53,9 @@
                   <box size ="${j1_l} ${j1_b} ${j1_h}" />
                   <limit lower="-${M_PI}" upper="${M_PI}" effort="1000" velocity="1000"/>
-                  <limit lower="-${M_PI/2}" upper="${M_PI/2}" effort="1000" velocity="1000"/>
+                  <limit lower="${j1_lower_lim}" upper="${j1_upper_lim}" effort="1000" velocity="1000"/>
                   <origin xyz="0 0 ${(base_length_2/2) + (j1_h /2)}" rpy="0 0 0"/>
                   <origin xyz="0 0 ${(j1_h/2) + j1_radius}" rpy="${M_PI/2} 0 0"/>
+                  <axis xyz="0 0 1" />
+                  <axis xyz="0 0 1" />
   </xacro:joint_arm>
   <xacro:joint_arm
@@ -66,7 +68,9 @@
                   <box size ="${j2_l} ${j2_b} ${j2_h}" />
                   <limit lower="0" upper="0" effort="0" velocity="0"/>
-                  <limit lower="-${M_PI/2}" upper="${M_PI/2}" effort="1000" velocity="1000"/>
+                  <limit lower="${j2_lower_lim}" upper="${j2_upper_lim}" effort="1000" velocity="1000"/>
                   <origin xyz="0 ${j1_radius + (j2_h /2)} 0" rpy="-${M_PI/2} -${M_PI} 0"/>
                   <origin xyz="0 0 ${(j2_h/2) + j2_radius}" rpy="0 ${M_PI/2} 0"/>
+                  <axis xyz="0 0 1" />
+                  <axis xyz="0 0 1" />
   </xacro:joint_arm>
   <xacro:joint_arm
@@ -79,7 +83,9 @@
                   <box size ="${j3_l} ${j3_b} ${j3_h}" />
                   <limit lower="0" upper="0" effort="0" velocity="0"/>
-                  <limit lower="-${M_PI/2}" upper="${M_PI/2}" effort="1000" velocity="1000"/>
+                  <limit lower="${j3_lower_lim}" upper="${j3_upper_lim}" effort="1000" velocity="1000"/>
                   <origin xyz="-${j2_radius + (j3_h /2)} 0 0" rpy="0 -${M_PI/2} 0"/>
                   <origin xyz="0 0 ${(j3_h/2) + j3_radius}" rpy="${M_PI/2} 0 ${M_PI}"/>
+                  <axis xyz="0 0 1" />
+                  <axis xyz="0 0 1" />
   </xacro:joint_arm>
   <xacro:joint_arm
@@ -92,7 +98,9 @@
                   <box size ="${j4_l} ${j4_b} ${j4_h}" />
                   <limit lower="0" upper="0" effort="0" velocity="0"/>
-                  <limit lower="-${M_PI/2}" upper="${M_PI/2}" effort="1000" velocity="1000"/>
+                  <limit lower="${j4_lower_lim}" upper="${j4_upper_lim}" effort="1000" velocity="1000"/>
                   <origin xyz="0 ${j3_radius + (j4_h /2)} 0" rpy="-${M_PI/2} -${M_PI} 0"/>
                   <origin xyz="0 0 ${(j4_h/2) + j4_radius}" rpy="0 ${M_PI/2} 0"/>
+                  <axis xyz="0 0 1" />
+                  <axis xyz="0 0 1" />
   </xacro:joint_arm>
   <xacro:joint_arm
@@ -105,7 +113,9 @@
                   <box size ="${j5_l} ${j5_b} ${j5_h}" />
                   <limit lower="0" upper="0" effort="0" velocity="0"/>
-                  <limit lower="-${M_PI/2}" upper="${M_PI/2}" effort="1000" velocity="1000"/>
+                  <limit lower="${j5_lower_lim}" upper="${j5_upper_lim}" effort="1000" velocity="1000"/>
                   <origin xyz="-${j4_radius + (j5_h /2)} 0 0" rpy="0 -${M_PI/2} 0"/>
                   <origin xyz="0 0 ${(j5_h/2) + j5_radius}" rpy="${M_PI/2} 0 ${M_PI}"/>
+                  <axis xyz="0 0 1" />
+                  <axis xyz="0 0 1" />
   </xacro:joint_arm>
  </xacro:macro>

File: src/rose20_description/cyton_gamma_1500/new/urdf/gripper/gripper.urdf.xacro (robot description, xacro)
@@ -23,22 +23,22 @@
   </xacro:macro>
   <!-- cyton_gamma_gripper: part 1 & 2 -->
- <xacro:macro name="cyton_gamma_gripper">
- <!-- Part 1 -->
- <xacro:part_gripper
+  <xacro:macro name="cyton_gamma_gripper">
+  <!-- Part 1 -->
+  <xacro:part_gripper
                   suffix=     "1"
                   parent=     "arm_link_cyl_5"
                   type =      "revolute">
                   <origin xyz="0 ${j5_radius + (gr1_1 /2)} 0" rpy="-${M_PI/2} ${M_PI/2} 0"/>
- 		  <limit lower="-${M_PI}" upper="${M_PI}" effort="1000" velocity="1000"/>
+ 		              <limit lower="${g1_lower_lim}" upper="${g1_upper_lim}" effort="1000" velocity="1000"/>
                   <box size ="${gr1_1} ${gr1_1} ${gr1_1}" />
- </xacro:part_gripper>
- <xacro:part_gripper
+  </xacro:part_gripper>
+  <xacro:part_gripper
                   suffix=     "2"
                   parent=     "gripper_link_1"
                   type =      "fixed">
                   <origin xyz="0 0 ${(gr1_1/2) + (gr1_2/2)}" rpy="0 0 0"/>
- 		  <limit lower="0" upper="0" effort="0" velocity="0"/>
+ 		              <limit lower="0" upper="0" effort="0" velocity="0"/>
                   <box size ="${gr1_2} ${gr1_2} ${gr1_2}" />
- </xacro:part_gripper>
+  </xacro:part_gripper>
   <!-- Part 2 -->
   <xacro:part_gripper
@@ -47,7 +47,7 @@
                   type =      "fixed">
                   <origin xyz="0 0 ${(gr1_2/2) + (gr2_1_h/2)}" rpy="0 0 0"/>
- 		  <limit lower="0" upper="0" effort="0" velocity="0"/>
+ 		              <limit lower="0" upper="0" effort="0" velocity="0"/>
                   <box size ="${gr2_1_l} ${gr2_1_b} ${gr2_1_h}" />
- </xacro:part_gripper>
+  </xacro:part_gripper>
   <xacro:part_gripper
                   suffix=     "4"
@@ -55,15 +55,15 @@
                   type =      "fixed">
                   <origin xyz="${gr2_1_l /4} ${(gr2_1_b /2) - (gr2_2_b /2)} ${(gr2_1_h/2) + (gr2_2_h/2)}" rpy="0 0 0"/>
- 		  <limit lower="0" upper="0" effort="0" velocity="0"/>
+ 		              <limit lower="0" upper="0" effort="0" velocity="0"/>
                   <box size ="${gr2_2_l} ${gr2_2_b} ${gr2_2_h}" />
- </xacro:part_gripper>
- <xacro:part_gripper
+  </xacro:part_gripper>
+  <xacro:part_gripper
                   suffix=     "5"
                   parent=     "gripper_link_3"
                   type =      "fixed">
                   <origin xyz="-${gr2_1_l /4} ${(gr2_1_b /2) - (gr2_2_b /2)} ${(gr2_1_h/2) + (gr2_2_h/2)}" rpy="0 0 0"/>
- 		  <limit lower="0" upper="0" effort="0" velocity="0"/>
+ 		              <limit lower="0" upper="0" effort="0" velocity="0"/>
                   <box size ="${gr2_2_l} ${gr2_2_b} ${gr2_2_h}" />
- </xacro:part_gripper>
- </xacro:macro>
+  </xacro:part_gripper>
+  </xacro:macro>
 </robot>

File: src/rose20_description/cyton_gamma_1500/new/urdf/properties/properties.urdf.xacro (robot description, xacro)
@@ -14,4 +14,6 @@
   <property name="j1_radius" value="0.036" />
   <property name="j1_length" value="0.08" />
+  <property name="j1_lower_lim" value="-2.6" />
+  <property name="j1_upper_lim" value="2.6" />
   <!--Joint 2-->
   <property name="j2_l" value="0.0445" />
@@ -20,4 +22,6 @@
   <property name="j2_radius" value="0.036" />
   <property name="j2_length" value="0.08" />
+  <property name="j2_lower_lim" value="-1.65" />
+  <property name="j2_upper_lim" value="1.65" />
   <!--Joint 3-->
   <property name="j3_l" value="0.0454" />
@@ -26,4 +30,6 @@
   <property name="j3_radius" value="0.036" />
   <property name="j3_length" value="0.08" />
+  <property name="j3_lower_lim" value="-1.60" />
+  <property name="j3_upper_lim" value="1.60" />
   <!--Joint 4-->
   <property name="j4_l" value="0.045" />
@@ -32,4 +38,6 @@
   <property name="j4_radius" value="0.0255" />
   <property name="j4_length" value="0.067" />
+  <property name="j4_lower_lim" value="-1.75" />
+  <property name="j4_upper_lim" value="1.75" />
   <!--Joint 5-->
   <property name="j5_l" value="0.045" />
@@ -38,8 +46,12 @@
   <property name="j5_radius" value="0.0245" />
   <property name="j5_length" value="0.045" />
+  <property name="j5_lower_lim" value="-1.90" />
+  <property name="j5_upper_lim" value="1.90" />
   <!--Gripper-->
   <!--Part 1-->
   <property name="gr1_1" value="0.04" />
   <property name="gr1_2" value="0.035" />
+  <property name="g1_lower_lim" value="-2.65" />
+  <property name="g1_upper_lim" value="2.65" />
   <!--Part 2-->
   <property name="gr2_1_l" value="0.065" />
